Commit message: xacro file works with camera and laserscan.. no laserscan or odom in rviz yet.. but soon to come!

File: src/robot_description/xacro/camera.xacro (robot description, xacro)
@@ -24,5 +24,5 @@
         <sensor name="camera" type="camera">
             <pose> 0 0 0 0 0 0 </pose>
-            <visualize>true</visualize>
+            <visualize>false</visualize>
             <update_rate>10</update_rate>
             <camera>
@@ -34,7 +34,4 @@
                 </image>
             </camera>
-            <plugin name="camera_controller" filename="libgazebo_ros_camera.so">
-                <frame_name>camera_link_optical</frame_name>
-            </plugin>
         </sensor>
     </gazebo>

File: src/robot_description/xacro/gazebo_control.xacro (robot description, xacro)
@@ -1,21 +1,19 @@
 <?xml version="1.0"?>
 <robot xmlns:xacro="http://www.ros.org/wiki/xacro" >
-  <gazebo>
-    <plugin name='gz::sim::systems::DiffDrive' filename='gz-sim-diff-drive-system'>
-      <!-- Wheel Information -->
-        <left_joint>left_wheel_joint</left_joint>
-        <right_joint>right_wheel_joint</right_joint>
-        <wheel_separation>0.44</wheel_separation>
-        <wheel_diameter>0.2</wheel_diameter>
-        <!-- Limits -->
-        <max_wheel_torque>200</max_wheel_torque>
-        <max_wheel_acceleration>10.0</max_wheel_acceleration>
-        <!-- Output -->
-        <odometry_frame>odom</odometry_frame>
-        <robot_base_frame>base_link</robot_base_frame>
-        <publish_odom>true</publish_odom>
-        <publish_odom_tf>true</publish_odom_tf>
-        <publish_wheel_tf>true</publish_wheel_tf>
-    </plugin>
-  </gazebo>
+    <gazebo>
+        <plugin
+            filename="gz-sim-diff-drive-system"
+            name="gz::sim::systems::DiffDrive">
+            <left_joint>left_wheel_joint</left_joint>
+            <right_joint>right_wheel_joint</right_joint>
+            <wheel_separation>0.440</wheel_separation>
+            <wheel_radius>0.1</wheel_radius>
+            <odom_publish_frequency>1</odom_publish_frequency>
+            <topic>/model/fejemis/cmd_vel</topic>
+            <odom_topic>/model/fejemis/odometry</odom_topic>
+            <tf_topic>/model/fejemis/tf</tf_topic>
+            <frame_id>odom</frame_id>
+            <child_frame_id>base_link</child_frame_id>
+        </plugin>
+    </gazebo>
 </robot>

File: src/robot_description/xacro/lidar.xacro (robot description, xacro)
@@ -1,9 +1,4 @@
 <?xml version="1.0"?>
 <robot xmlns:xacro="http://www.ros.org/wiki/xacro" >
-    <joint name="laser_joint" type="fixed">
-        <parent link="chassis"/>
-        <child link="laser_frame"/>
-        <origin xyz="0.07 0 0.329" rpy="0 0 0"/>
-    </joint>
     <link name="laser_frame">
         <visual>
@@ -22,31 +17,39 @@
         </xacro:inertial_cylinder>
     </link>
-    <sensor name='gpu_lidar' type='gpu_lidar'>"
-        <pose relative_to='laser_frame'>0 0 0 0 0 0</pose>
-        <topic>lidar</topic>
-        <update_rate>10</update_rate>
-        <ray>
-            <scan>
-                <horizontal>
-                    <samples>360</samples>
-                    <resolution>1</resolution>
-                    <min_angle>-1.396263</min_angle>
-                    <max_angle>1.396263</max_angle>
-                </horizontal>
-                <vertical>
-                    <samples>1</samples>
-                    <resolution>0.01</resolution>
-                    <min_angle>0</min_angle>
-                    <max_angle>0</max_angle>
-                </vertical>
-            </scan>
-            <range>
-                <min>0.08</min>
-                <max>15.0</max>
-                <resolution>0.01</resolution>
-            </range>
-        </ray>
-        <always_on>1</always_on>
-        <visualize>true</visualize>
-    </sensor>
+    <joint name="laser_joint" type="fixed">
+        <parent link="chassis"/>
+        <child link="laser_frame"/>
+        <origin xyz="0.07 0 0.329" rpy="0 0 0"/>
+    </joint>
+    <gazebo reference="laser_frame">
+        <material>Gazebo/Black</material>
+        <sensor name='gpu_lidar' type='gpu_lidar'>"
+                <pose relative_to='chassis'>0.15 0 0.329 0 0.06 0</pose>
+                <topic>lidar</topic>
+                <update_rate>10</update_rate>
+                <ray>
+                    <scan>
+                        <horizontal>
+                            <samples>640</samples>
+                            <resolution>1</resolution>
+                            <min_angle>-3.14</min_angle>
+                            <max_angle>3.14</max_angle>
+                        </horizontal>
+                        <vertical>
+                            <samples>1</samples>
+                            <resolution>0.01</resolution>
+                            <min_angle>0</min_angle>
+                            <max_angle>0</max_angle>
+                        </vertical>
+                    </scan>
+                    <range>
+                        <min>0.1</min>
+                        <max>15.0</max>
+                        <resolution>0.015</resolution>
+                    </range>
+                </ray>
+                <always_on>1</always_on>
+                <visualize>true</visualize>
+            </sensor>
+    </gazebo>
 </robot>

File: src/robot_description/xacro/robot.urdf.xacro (robot description, xacro)
@@ -1,15 +1,14 @@
 <?xml version="1.0"?>
-<robot xmlns:xacro="http://www.ros.org/wiki/xacro"  name="fejemis">
-    <!-- <xacro:arg name="use_ros2_control" default="true"/> -->
+<robot xmlns:xacro="http://www.ros.org/wiki/xacro"  name="robot">
+    <xacro:arg name="use_ros2_control" default="false"/>
     <xacro:include filename="robot_core.xacro" />
-    <!-- <xacro:if value="$(arg use_ros2_control)">
+    <xacro:if value="$(arg use_ros2_control)">
     <xacro:include filename="ros2_control.xacro" />
     </xacro:if>
     <xacro:unless value="$(arg use_ros2_control)">
     <xacro:include filename="gazebo_control.xacro" />
-    </xacro:unless> -->
-    <xacro:include filename="gazebo_control.xacro" />
+    </xacro:unless>
     <xacro:include filename="lidar.xacro" />
-    <!-- <xacro:include filename="camera.xacro" /> -->
+    <xacro:include filename="camera.xacro" />
     <!-- xacro:include filename="depth_camera.xacro" /> -->
 </robot>

File: src/robot_description/xacro/robot_core.xacro (robot description, xacro)
@@ -58,7 +58,7 @@
         </xacro:inertial_box> -->
     </link>
-    <!-- <gazebo reference="chassis">
+    <gazebo reference="chassis">
         <material>Gazebo/Yellow</material>
-    </gazebo> -->
+    </gazebo>
     <!-- LEFT WHEEL LINK -->
     <joint name="left_wheel_joint" type="continuous">
@@ -84,7 +84,7 @@
         </xacro:inertial_cylinder>
     </link>
-    <!-- <gazebo reference="left_wheel">
+    <gazebo reference="left_wheel">
         <material>Gazebo/Black</material>
-    </gazebo> -->
+    </gazebo>
     <!-- RIGHT WHEEL LINK -->
     <joint name="right_wheel_joint" type="continuous">
@@ -110,7 +110,7 @@
         </xacro:inertial_cylinder>
     </link>
-    <!-- <gazebo reference="right_wheel">
+    <gazebo reference="right_wheel">
         <material>Gazebo/Black</material>
-    </gazebo> -->
+    </gazebo>
     <!-- CASTER WHEEL LINK -->
     <joint name="caster_wheel_joint" type="fixed">
@@ -135,8 +135,8 @@
         </xacro:inertial_sphere>
     </link>
-    <!-- <gazebo reference="caster_wheel">
+    <gazebo reference="caster_wheel">
         <material>Gazebo/White</material>
         <mu1 value="0.001"/>
         <mu2 value="0.001"/>
-    </gazebo> -->
+    </gazebo>
 </robot>

File: src/robot_description/xacro/ros2_control.xacro (robot description, xacro)
@@ -3,5 +3,12 @@
     <ros2_control name="RealRobot" type="system">
         <hardware>
-            <plugin>gz_ros2_control/GazeboSimSystem</plugin>
+            <plugin>diffdrive_arduino/DiffDriveArduino</plugin>
+            <param name="left_wheel_name">left_wheel_joint</param>
+            <param name="right_wheel_name">right_wheel_joint</param>
+            <param name="loop_rate">30</param>
+            <param name="device">/dev/ttyACM1</param>
+            <param name="baud_rate">115200</param>
+            <param name="timeout">1000</param>
+            <param name="enc_counts_per_rev">3436</param>
         </hardware>
         <joint name="left_wheel_joint">
@@ -43,18 +50,8 @@
         </joint>
     </ros2_control> -->
-    <!-- <gazebo>
+    <gazebo>
     <plugin filename="libgazebo_ros2_control.so" name="gazebo_ros2_control">
-        <parameters>$(find robot_simulation)/config/controller.yaml</parameters>
+        <parameters>$(find fejemis_sim)/config/my_controller.yaml</parameters>
     </plugin>
     </gazebo>
-    <hardware>
-            <plugin>diffdrive_arduino/DiffDriveArduino</plugin>
-            <param name="left_wheel_name">left_wheel_joint</param>
-            <param name="right_wheel_name">right_wheel_joint</param>
-            <param name="loop_rate">30</param>
-            <param name="device">/dev/ttyACM1</param>
-            <param name="baud_rate">115200</param>
-            <param name="timeout">1000</param>
-            <param name="enc_counts_per_rev">3436</param>
-    </hardware> -->
 </robot>

Commit message: Nu har jeg fået odom til at virke og nu skal lidar bare også virke i rviz2

File: src/robot_description/xacro/camera.xacro (robot description, xacro)
@@ -1,4 +1,4 @@
 <?xml version="1.0"?>
-<robot xmlns:xacro="http://www.ros.org/wiki/xacro"  name="robot">
+<robot xmlns:xacro="http://www.ros.org/wiki/xacro"  name="fejemis">
     <joint name="camera_joint" type="fixed">
         <parent link="chassis"/>

File: src/robot_description/xacro/depth_camera.xacro (robot description, xacro)
@@ -1,4 +1,4 @@
 <?xml version="1.0"?>
-<robot xmlns:xacro="http://www.ros.org/wiki/xacro"  name="robot">
+<robot xmlns:xacro="http://www.ros.org/wiki/xacro"  name="fejemis">
     <joint name="camera_joint" type="fixed">
         <parent link="chassis"/>

File: src/robot_description/xacro/gazebo_control.xacro (robot description, xacro)
@@ -9,10 +9,10 @@
             <wheel_separation>0.440</wheel_separation>
             <wheel_radius>0.1</wheel_radius>
-            <odom_publish_frequency>1</odom_publish_frequency>
+            <odom_publish_frequency>10</odom_publish_frequency>
             <topic>/model/fejemis/cmd_vel</topic>
             <odom_topic>/model/fejemis/odometry</odom_topic>
             <tf_topic>/model/fejemis/tf</tf_topic>
-            <frame_id>odom</frame_id>
-            <child_frame_id>base_link</child_frame_id>
+            <frame_id>/odom</frame_id>
+            <child_frame_id>/base_link</child_frame_id>
         </plugin>
     </gazebo>

File: src/robot_description/xacro/robot.urdf.xacro (robot description, xacro)
@@ -1,4 +1,4 @@
 <?xml version="1.0"?>
-<robot xmlns:xacro="http://www.ros.org/wiki/xacro"  name="robot">
+<robot xmlns:xacro="http://www.ros.org/wiki/xacro"  name="fejemis">
     <xacro:arg name="use_ros2_control" default="false"/>
     <xacro:include filename="robot_core.xacro" />

File: src/robot_description/xacro/robot_core.xacro (robot description, xacro)
@@ -1,5 +1,6 @@
 <?xml version="1.0"?>
-<robot xmlns:xacro="http://www.ros.org/wiki/xacro" >
+<robot xmlns:xacro="http://www.ros.org/wiki/xacro">
     <xacro:include filename="inertial_macros.xacro"/>
+    <!-- Define Materials -->
     <material name="white">
         <color rgba="1 1 1 1" />
@@ -20,8 +21,7 @@
         <color rgba="0.616 0.616 0.616 1"/>
     </material>
-    <!-- BASE LINK -->
-    <link name="base_link">
-    </link>
-    <!-- BASE FOOTPRINT LINK-->
+    <!-- Base Link -->
+    <link name="base_link"></link>
+    <!-- Base Footprint Link -->
     <joint name="base_footprint_joint" type="fixed">
         <parent link="base_link"/>
@@ -30,5 +30,5 @@
     </joint>
     <link name="base_footprint"></link>
-    <!-- CHASSIS LINK -->
+    <!-- Chassis Link -->
     <joint name="chassis_joint" type="fixed">
         <parent link="base_footprint"/>
@@ -44,22 +44,18 @@
             <material name="yellow"/>
         </visual>
-        <!-- <collision>
+        <collision>
             <origin xyz="0.426 0 0.130"/>
             <geometry>
-                <box size="0.01 0.01 0.01"/>
                 <box size="0.810 0.500 0.259"/>
             </geometry>
-        </collision> -->
+        </collision>
         <xacro:inertial_box mass="0.3" x="0.810" y="0.500" z="0.259">
             <origin xyz="0.426 0 0.130" rpy="0 0 0"/>
         </xacro:inertial_box>
-        <!-- <xacro:inertial_box mass="1" x="0.810" y="0.500" z="0.259">
-            <origin xyz="0 0 0" rpy="0 0 0"/>
-        </xacro:inertial_box> -->
     </link>
     <gazebo reference="chassis">
         <material>Gazebo/Yellow</material>
     </gazebo>
-    <!-- LEFT WHEEL LINK -->
+    <!-- Left Wheel Link -->
     <joint name="left_wheel_joint" type="continuous">
         <parent link="base_footprint"/>
@@ -87,5 +83,5 @@
         <material>Gazebo/Black</material>
     </gazebo>
-    <!-- RIGHT WHEEL LINK -->
+    <!-- Right Wheel Link -->
     <joint name="right_wheel_joint" type="continuous">
         <parent link="base_footprint"/>
@@ -113,5 +109,5 @@
         <material>Gazebo/Black</material>
     </gazebo>
-    <!-- CASTER WHEEL LINK -->
+    <!-- Caster Wheel Link -->
     <joint name="caster_wheel_joint" type="fixed">
         <parent link="chassis"/>

File: src/robot_description/xacro/ros2_control.xacro (robot description, xacro)
@@ -1,5 +1,5 @@
 <?xml version="1.0"?>
 <robot xmlns:xacro="http://www.ros.org/wiki/xacro" >
-    <ros2_control name="RealRobot" type="system">
+    <ros2_control name="fejemis" type="system">
         <hardware>
             <plugin>diffdrive_arduino/DiffDriveArduino</plugin>
