Commit message: Ros2_control is now working and can control the robot with that

File: src/robot_description/xacro/lidar.xacro (robot description, xacro)
@@ -1,5 +1,5 @@
 <?xml version="1.0"?>
 <robot xmlns:xacro="http://www.ros.org/wiki/xacro" >
-    <link name="laser_frame">
+    <link name="lidar_frame">
         <visual>
             <geometry>
@@ -19,37 +19,37 @@
     <joint name="laser_joint" type="fixed">
         <parent link="chassis"/>
-        <child link="laser_frame"/>
+        <child link="lidar_frame"/>
         <origin xyz="0.07 0 0.329" rpy="0 0 0"/>
     </joint>
-    <gazebo reference="laser_frame">
+    <gazebo reference="lidar_frame">
         <material>Gazebo/Black</material>
-        <sensor name='gpu_lidar' type='gpu_lidar'>"
-                <pose relative_to='chassis'>0.15 0 0.329 0 0.06 0</pose>
-                <topic>lidar</topic>
-                <update_rate>10</update_rate>
-                <ray>
-                    <scan>
-                        <horizontal>
-                            <samples>640</samples>
-                            <resolution>1</resolution>
-                            <min_angle>-3.14</min_angle>
-                            <max_angle>3.14</max_angle>
-                        </horizontal>
-                        <vertical>
-                            <samples>1</samples>
-                            <resolution>0.01</resolution>
-                            <min_angle>0</min_angle>
-                            <max_angle>0</max_angle>
-                        </vertical>
-                    </scan>
-                    <range>
-                        <min>0.1</min>
-                        <max>15.0</max>
-                        <resolution>0.015</resolution>
-                    </range>
-                </ray>
-                <always_on>1</always_on>
-                <visualize>true</visualize>
-            </sensor>
+        <sensor name='laser_scanner' type='gpu_lidar'>"
+            <pose relative_to='chassis'>0.15 0 0.329 0 0.06 0</pose>
+            <topic>lidar</topic>
+            <update_rate>30</update_rate>
+            <ray>
+                <scan>
+                    <horizontal>
+                        <samples>720</samples>
+                        <resolution>1</resolution>
+                        <min_angle>-3.14</min_angle>
+                        <max_angle>3.14</max_angle>
+                    </horizontal>
+                    <vertical>
+                        <samples>1</samples>
+                        <resolution>0.1</resolution>
+                        <min_angle>0.01</min_angle>
+                        <max_angle>3.14</max_angle>
+                    </vertical>
+                </scan>
+                <range>
+                    <min>0.1</min>
+                    <max>15.0</max>
+                    <resolution>0.01</resolution>
+                </range>
+            </ray>
+            <always_on>1</always_on>
+            <visualize>true</visualize>
+        </sensor>
     </gazebo>
 </robot>

File: src/robot_description/xacro/robot.urdf.xacro (robot description, xacro)
@@ -1,5 +1,5 @@
 <?xml version="1.0"?>
 <robot xmlns:xacro="http://www.ros.org/wiki/xacro"  name="fejemis">
-    <xacro:arg name="use_ros2_control" default="false"/>
+     <xacro:arg name="use_ros2_control" default="false"/> <!-- #denne her driller mig meget... Den køre hvis den er false, men ikke i true-->
     <xacro:include filename="robot_core.xacro" />
     <xacro:if value="$(arg use_ros2_control)">
@@ -11,4 +11,6 @@
     <xacro:include filename="lidar.xacro" />
     <xacro:include filename="camera.xacro" />
+    <!-- <xacro:include filename="ros2_control.xacro" /> -->
+    <!-- <xacro:include filename="gazebo_control.xacro" /> -->
     <!-- xacro:include filename="depth_camera.xacro" /> -->
 </robot>

File: src/robot_description/xacro/robot_core.xacro (robot description, xacro)
@@ -32,5 +32,5 @@
     <!-- Chassis Link -->
     <joint name="chassis_joint" type="fixed">
-        <parent link="base_footprint"/>
+        <parent link="base_link"/>
         <child link="chassis"/>
         <origin xyz="-0.1 0 0"/>
@@ -59,5 +59,5 @@
     <!-- Left Wheel Link -->
     <joint name="left_wheel_joint" type="continuous">
-        <parent link="base_footprint"/>
+        <parent link="base_link"/>
         <child link="left_wheel"/>
         <origin xyz="0 0.220 0" rpy="-${pi/2} 0 0" />
@@ -85,5 +85,5 @@
     <!-- Right Wheel Link -->
     <joint name="right_wheel_joint" type="continuous">
-        <parent link="base_footprint"/>
+        <parent link="base_link"/>
         <child link="right_wheel"/>
         <origin xyz="0 -0.220 0" rpy="${pi/2} 0 0" />

File: src/robot_description/xacro/ros2_control.xacro (robot description, xacro)
@@ -1,5 +1,5 @@
 <?xml version="1.0"?>
 <robot xmlns:xacro="http://www.ros.org/wiki/xacro" >
-    <ros2_control name="fejemis" type="system">
+    <!-- <ros2_control name="fejemis" type="system">
         <hardware>
             <plugin>diffdrive_arduino/DiffDriveArduino</plugin>
@@ -28,8 +28,8 @@
             <state_interface name="position"/>
         </joint>
-    </ros2_control>
-   <!-- <ros2_control name="GazeboSystem" type="system">
+    </ros2_control> -->
+   <ros2_control name="GazeboSimSystem" type="system">
         <hardware>
-            <plugin>gazebo_ros2_control/GazeboSystem</plugin>
+            <plugin>gz_ros2_control/GazeboSimSystem</plugin>
         </hardware>
         <joint name="left_wheel_joint">
@@ -49,9 +49,9 @@
             <state_interface name="position" />
         </joint>
-    </ros2_control> -->
+    </ros2_control>
     <gazebo>
-    <plugin filename="libgazebo_ros2_control.so" name="gazebo_ros2_control">
-        <parameters>$(find fejemis_sim)/config/my_controller.yaml</parameters>
-    </plugin>
+        <plugin filename="libgz_ros2_control-system.so" name="gz_ros2_control::GazeboSimROS2ControlPlugin">
+            <parameters>$(find robot_description)/config/my_controllers.yaml</parameters>
+        </plugin>
     </gazebo>
 </robot>
